File: hardware/plant_monitor.kicad_pcb (KiCad board)
At the start: 4 copper layers, 74.8 x 84.2 mm, 208 parts, among them J1 Conn_01x03_Female, J2 Conn_01x03_Male, J3 Conn_01x06_Male, Q1 BSS84, Q2 BSS84, Q3 BSS138, U1 MCP9808T-E_MS, U2 SHTC3, U3 SI1133-AA00-GMR, U4 MS563702BA03-50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

Commit message: wip 2
Parts:
- removed R88: 0R, Resistor_SMD:R_0402_1005Metric
- U9: footprint sweet:XCVR_WSSFM10R1AT -> plant_monitor:XCVR_WSSFM10R1AT_HANDSOLDER
- moved R99 16.8 mm to (134.9, 109.5), turned to 180 degrees
- moved ANT1 14.4 mm to (120.4, 90.1), turned to 0 degrees
- moved R89 14.1 mm to (125.2, 90.1), turned to 0 degrees
- moved R96 13.8 mm to (132.9, 109.5), turned to 0 degrees
- moved R93 13.1 mm to (132.9, 108.5), turned to 0 degrees
- moved R91 12.6 mm to (132.9, 102.0), turned to 90 degrees
- moved R92 12.4 mm to (132.9, 107.5), turned to 180 degrees
- moved R97 12.2 mm to (113.0, 105.5), turned to 180 degrees
- moved L3 11.5 mm to (117.0, 95.9)
- moved C34 11.4 mm to (117.5, 97.5)
- moved R90 11.4 mm to (117.0, 92.9)
- moved R87 11.4 mm to (117.5, 94.4)
- moved TP29 11.4 mm to (121.9, 111.8), turned to 0 degrees
- moved FB4 10.9 mm to (133.5, 97.6), turned to 0 degrees
- moved TP30 10.8 mm to (132.1, 104.1), turned to 90 degrees
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Connections:
- R87 pad 2: Net-(R87-Pad2) -> Net-(ANT1-Pad1)
- R90 pad 2: Net-(R87-Pad2) -> Net-(ANT1-Pad1)
Routing:
- net Net-(R98-Pad1): track 5.73 -> 29.2 mm, vias 1 -> 2
- net Net-(D7-Pad2): track 23.1 -> 2.08 mm, vias 3 -> 0
- net Net-(R97-Pad1): track 3.32 -> 21.4 mm, vias 1 -> 2
- net Net-(D6-Pad2): track 20.1 -> 2.10 mm, vias 3 -> 0
- net /mcu/SIGFOX_RST_N: track 54.3 -> 72.1 mm, vias 3 -> 5
- net Net-(R95-Pad2): track 1.64 -> 17.6 mm, vias 0 -> 2
- net /mcu/SIGFOX_TX: track 22.4 -> 37.4 mm, vias 3 -> 4
- net /mcu/SIGFOX_RX: track 30.5 -> 45.1 mm, vias 4 -> 5
- net Net-(R94-Pad2): track 1.64 -> 15.4 mm, vias 0 -> 2
- net /mcu/SIGFOX_WAKE_UP: track 40.4 -> 46.5 mm
- net GND: track 28.4 -> 34.4 mm, vias 18 -> 22
- net Net-(TP31-Pad1): track 3.08 -> 7.99 mm
- net Net-(ANT1-Pad1): track 0.00 -> 3.96 mm
- net Net-(C34-Pad1): track 0.00 -> 2.65 mm
- net Net-(TP33-Pad1): track 0.00 -> 2.55 mm, vias 0 -> 1
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Other:
- net class Default: clearance 0.2 -> 0.15
- rule trace_clearance: 0.2 -> 0.15
